Commit message: update model

File: src/simulation/urdf/simple.urdf (robot description, URDF)
Before this commit: robot simple, 2 links, 1 joints
Links:
- removed link right_back_wheel
- added link front_wheel, mass 1; collision sphere radius=0.05; visual sphere radius=0.05
- added link left_wheel, mass 1; collision cylinder length=0.1 radius=0.1; visual cylinder length=0.1 radius=0.1
- added link right_wheel, mass 1; collision cylinder length=0.1 radius=0.1; visual cylinder length=0.1 radius=0.1
- link base_link: mass 10 -> 5
Joints:
- removed joint back_right_wheel_to_base
- added joint base_to_front_wheel: type continuous, parent base_link, child front_wheel, origin xyz=0 0.2 -0.05 rpy=0 0 0, axis 1 0 0
- added joint base_to_left_wheel: type continuous, parent base_link, child left_wheel, origin xyz=0.18 -0.2 0.0 rpy=0.0 1.5707 0.0, axis 0 0 1
- added joint base_to_right_wheel: type continuous, parent base_link, child right_wheel, origin xyz=-0.18 -0.2 0.0 rpy=0.0 1.5707 0.0, axis 0 0 1
